Commit message: fixed names

File: mm_arena/common/robots/youbot.urdf.xacro (robot description, xacro)
@@ -40,4 +40,4 @@
     <origin xyz="0 0 0" rpy="0 0 0" />
   </xacro:youbot_gripper>
-  <youbot_kinect/>
+  <kinect_gazebo/>
 </robot>

File: mm_arena/common/sensors/kinect.urdf.xacro (robot description, xacro)
@@ -4,5 +4,5 @@
   <include filename="$(find mm_arena)/common/sensors/kinect.gazebo.urdf.xacro"/>
   <include filename="$(find mm_arena)/common/sensors/kinect.config.urdf.xacro" />
-<xacro:macro name="kinect">
+<xacro:macro name="kinect_gazebo">
   <joint name="base_camera_joint" type="fixed">
     <origin xyz="${kinect_position_x} ${kinect_position_y} ${kinect_position_z}"
