Commit message: changed cube size from 0.1m to 0.04
change bluecube.urdf
change greencube.urdf
change redcube.urdf

File: mm_arena/common/objects/bluecube.urdf (robot description, URDF)
Before this commit: robot bluecube_model, 2 links, 1 joints
Links:
- link bluecube1: geometry collision box size=0.04 0.04 0.04; visual box size=0.04 0.04 0.04

File: mm_arena/common/objects/greencube.urdf (robot description, URDF)
Before this commit: robot greencube_model, 2 links, 1 joints
Links:
- link greencube1: geometry collision box size=0.04 0.04 0.04; visual box size=0.04 0.04 0.04

File: mm_arena/common/objects/redcube.urdf (robot description, URDF)
Before this commit: robot redcube_model, 2 links, 1 joints
Links:
- link redcube1: geometry collision box size=0.04 0.04 0.04; visual box size=0.04 0.04 0.04
