Commit message: changed cubes

File: mm_arena/common/objects/base.urdf (robot description, URDF)
Before this commit: robot bluecube_model, 2 links, 1 joints
Links:
- removed link bluecube1
- added link base, mass 0.1; collision box size=0.2 0.2 0.08; visual box size=0.2 0.2 0.08
Joints:
- joint cube1_joint: child bluecube1 -> base; origin xyz=0 0.0 0.02 rpy=0 0 0 -> xyz=0 0.0 0.05 rpy=0 0 0

File: mm_arena/common/objects/greenbase.urdf (robot description, URDF)
Before this commit: robot bluecube_model, 2 links, 1 joints
Links:
- removed link bluecube1
- added link greenbase, mass 0.1; collision box size=0.2 0.2 0.10; visual box size=0.2 0.2 0.10
Joints:
- joint cube1_joint: child bluecube1 -> greenbase; origin xyz=0 0.0 0.02 rpy=0 0 0 -> xyz=0 0.0 0.05 rpy=0 0 0

File: mm_arena/common/objects/greencube.urdf (robot description, URDF)
Before this commit: robot greencube_model, 2 links, 1 joints
Joints:
- joint cube1_joint: origin xyz=0.0 0.0 0.05 rpy=0 0 0 -> xyz=0.0 0.0 0.02 rpy=0 0 0

File: mm_arena/common/objects/redbase.urdf (robot description, URDF)
Before this commit: robot bluecube_model, 2 links, 1 joints
Links:
- removed link bluecube1
- added link redbase, mass 1.1; collision box size=0.2 0.2 0.10; visual box size=0.2 0.2 0.10
Joints:
- joint cube1_joint: child bluecube1 -> redbase; origin xyz=0 0.0 0.02 rpy=0 0 0 -> xyz=0 0.0 0.05 rpy=0 0 0

File: mm_arena/common/objects/redcube.urdf (robot description, URDF)
Before this commit: robot redcube_model, 2 links, 1 joints
Joints:
- joint cube1_joint: origin xyz=0 0.0 0.05 rpy=0 0 0 -> xyz=0 0.0 0.02 rpy=0 0 0

File: mm_arena/common/robots/youbot.urdf.xacro (robot description, xacro)
@@ -16,5 +16,6 @@
   <include filename="$(find mm_arena)/common/sensors/kinect.urdf.xacro" />
   <!-- youbot gripper -->
-  <include filename="$(find youbot_description)/urdf/youbot_gripper/gripper.urdf.xacro" />
+  <!--<include filename="$(find youbot_description)/urdf/youbot_gripper/gripper.urdf.xacro" />-->
+  <include filename="$(find mm_arena)/common/robots/gripper.urdf.xacro" />
   <!-- generic simulator_gazebo plugins for starting mechanism control, ros time, ros battery -->
   <include filename="$(find youbot_description)/gazebo/gazebo.urdf.xacro" />

File: mm_arena/common/sensors/kinect.gazebo.urdf.xacro (robot description, xacro)
@@ -7,11 +7,11 @@
       <imageSize>640 480</imageSize>
       <hfov>57</hfov>
-      <nearClip>0.1</nearClip>
+      <nearClip>0.45</nearClip>
       <farClip>5</farClip>
-      <updateRate>20.0</updateRate>
+      <updateRate>1.0</updateRate>
       <baseline>0.2</baseline>
       <controller:gazebo_ros_openni_kinect name="kinect_camera_controller" plugin="libgazebo_ros_openni_kinect.so">
         <alwaysOn>true</alwaysOn>
-        <updateRate>20.0</updateRate>
+        <updateRate>1.0</updateRate>
         <imageTopicName>/camera/image_raw</imageTopicName>
         <pointCloudTopicName>/camera/depth/points</pointCloudTopicName>
